File: uClouds_002-frontpanelV7.brd (EAGLE design)
At the start: 40.6 x 128.5 mm, 1 part

Commit message: final final ready for print
BAckside included
Parts:
- added E$2: (no value), bfl:OSHW1
- moved E$1 0.25 mm to (16.8, 2.54)
Routing:
- added copper zone on layer 16, net S$10
- added copper zone on layer 16, net S$6
- added copper zone on layer 16, net S$7
- added copper zone on layer 16, net S$8
- added copper zone on layer 16, net S$9
Other:
- board text added: "Creative Commons CC-BY-SA-3.0"
- board text added: "Custom frontpanel by monomanic Rotterdam"
- board text added: "Too weird to live, too rare to die"
- board text added: "original design by Mutable Instruments"
- board text added: "uClouds design by Jason H. J. Lim"
